Commit message: add lidar

File: Desktop/software_engineering_robotics_Udacity/projects/catkin_ws_chase_ball/src/av_robot/urdf/robot.xacro (robot description, xacro)
@@ -26,4 +26,10 @@
         <parent link="chassis"/>
         <child link="camera"/>
+        <axis xyz="0 1 0" rpy="0 0 0"/>
+    </joint>
+    <joint name="hokuyo_joint" type="fixed">
+        <origin xyz="0.15 0 0.1" rpy="0 0 0"/>
+        <parent link="chassis"/>
+        <child link="hokuyo"/>
         <axis xyz="0 1 0" rpy="0 0 0"/>
     </joint>
@@ -144,3 +150,24 @@
         </visual>
     </link>
+    <link name="hokuyo">
+        <inertial>
+            <mass value="1e-5"/>
+            <origin xyz="0 0 0" rpy="0 0 0"/>
+            <inertia
+                    ixx="1e-6" ixy="0" ixz="0" iyy="1e-6" iyz="0" izz="1e-6"
+            />
+        </inertial>
+        <collision name="hokuyo_collision">
+            <origin xyz="0 0 0" rpy="0 0 0"/>
+            <geometry>
+                <box size="0.1 0.1 0.1"/>
+            </geometry>
+        </collision>
+        <visual name="hokuyo_visual">
+            <origin xyz="0 0 0" rpy="0 0 0"/>
+            <geometry>
+                <mesh filename = "package://av_robot/meshes/hokuyo.dae"/>
+            </geometry>
+        </visual>
+    </link>
 </robot>

Commit message: add materials to the robot

File: Desktop/software_engineering_robotics_Udacity/projects/catkin_ws_chase_ball/src/av_robot/urdf/robot.xacro (robot description, xacro)
@@ -33,4 +33,7 @@
         <child link="hokuyo"/>
         <axis xyz="0 1 0" rpy="0 0 0"/>
+        <gazebo reference="right_wheel">
+            <material>Gazebo/Green</material>
+        </gazebo>
     </joint>
     <link name='chassis'>
@@ -171,3 +174,15 @@
         </visual>
     </link>
+    <gazebo reference="left_wheel">
+        <material>Gazebo/Green</material>
+    </gazebo>
+    <gazebo reference="right_wheel">
+        <material>Gazebo/Green</material>
+    </gazebo>
+    <gazebo reference="chassis">
+        <material>Gazebo/Blue</material>
+    </gazebo>
+    <gazebo reference="camera">
+        <material>Gazebo/Red</material>
+    </gazebo>
 </robot>

Commit message: ball cheaser completed

File: Desktop/software_engineering_robotics_Udacity/projects/catkin_ws_chase_ball/src/av_robot/urdf/robot.xacro (robot description, xacro)
@@ -8,5 +8,5 @@
     </joint>
     <joint name="left_wheel_hinge" type="continuous">
-        <origin xyz="0 0.15 0" rpy="0 0 0"/>
+        <origin xyz="0 0.3 0" rpy="0 0 0"/>
         <child link="left_wheel"/>
         <parent link="chassis"/>
@@ -16,5 +16,5 @@
     </joint>
     <joint name="right_wheel_hinge" type="continuous">
-        <origin xyz="0 -0.15 0" rpy="0 0 0"/>
+        <origin xyz="0 -0.3 0" rpy="0 0 0"/>
         <child link="right_wheel"/>
         <parent link="chassis"/>
@@ -24,5 +24,5 @@
     </joint>
     <joint name="camera_joint" type="fixed">
-        <origin xyz="0.2 0 0" rpy="0 0 0"/>
+        <origin xyz="0.4 0 0" rpy="0 0 0"/>
         <parent link="chassis"/>
         <child link="camera"/>
@@ -52,5 +52,5 @@
             <origin xyz="0 0 0" rpy=" 0 0 0"/>
             <geometry>
-                <box size=".4 .2 .1"/>
+                <box size=".8 .4 .2"/>
             </geometry>
         </collision>
@@ -58,29 +58,29 @@
             <origin xyz="0 0 0" rpy=" 0 0 0"/>
             <geometry>
-                <box size=".4 .2 .1"/>
+                <box size=".8 .4 .2"/>
             </geometry>
         </visual>
         <collision name='back_caster_collision'>
-            <origin xyz="-0.15 0 -0.05" rpy=" 0 0 0"/>
+            <origin xyz="-0.3 0 -0.05" rpy=" 0 0 0"/>
             <geometry>
-                <sphere radius="0.0499"/>
+                <sphere radius="0.099"/>
             </geometry>
         </collision>
         <visual name='back_caster_visual'>
-            <origin xyz="-0.15 0 -0.05" rpy=" 0 0 0"/>
+            <origin xyz="-0.3 0 -0.1" rpy=" 0 0 0"/>
             <geometry>
-                <sphere radius="0.05"/>
+                <sphere radius="0.1"/>
             </geometry>
         </visual>
         <collision name='front_caster_collision'>
-            <origin xyz="0.15 0 -0.05" rpy=" 0 0 0"/>
+            <origin xyz="0.3 0 -0.1" rpy=" 0 0 0"/>
             <geometry>
-                <sphere radius="0.0499"/>
+                <sphere radius="0.099"/>
             </geometry>
         </collision>
         <visual name='front_caster_visual'>
-            <origin xyz="0.15 0 -0.05" rpy=" 0 0 0"/>
+            <origin xyz="0.3 0 -0.1" rpy=" 0 0 0"/>
             <geometry>
-                <sphere radius="0.05"/>
+                <sphere radius="0.1"/>
             </geometry>
         </visual>
@@ -99,5 +99,5 @@
             <origin xyz="0 0 0" rpy="0 1.5707 1.5707"/>
             <geometry>
-                <cylinder radius="0.1" length="0.05"/>
+                <cylinder radius="0.2" length="0.05"/>
             </geometry>
         </collision>
@@ -105,5 +105,5 @@
             <origin xyz="0 0 0" rpy="0 1.5707 1.5707"/>
             <geometry>
-                <cylinder radius="0.1" length="0.05"/>
+                <cylinder radius="0.2" length="0.05"/>
             </geometry>
         </visual>
@@ -122,5 +122,5 @@
             <origin xyz="0 0 0" rpy="0 1.5707 1.5707"/>
             <geometry>
-                <cylinder radius="0.1" length="0.05"/>
+                <cylinder radius="0.2" length="0.05"/>
             </geometry>
         </collision>
@@ -128,5 +128,5 @@
             <origin xyz="0 0 0" rpy="0 1.5707 1.5707"/>
             <geometry>
-                <cylinder radius="0.1" length="0.05"/>
+                <cylinder radius="0.2" length="0.05"/>
             </geometry>
         </visual>
@@ -176,14 +176,14 @@
     </link>
     <gazebo reference="left_wheel">
-        <material>Gazebo/Green</material>
+        <material>Gazebo/Orange</material>
     </gazebo>
     <gazebo reference="right_wheel">
-        <material>Gazebo/Green</material>
+        <material>Gazebo/Orange</material>
     </gazebo>
     <gazebo reference="chassis">
+        <material>Gazebo/Red</material>
+    </gazebo>
+    <gazebo reference="camera">
         <material>Gazebo/Blue</material>
     </gazebo>
-    <gazebo reference="camera">
-        <material>Gazebo/Red</material>
-    </gazebo>
 </robot>

Commit message: modifications

File: Desktop/software_engineering_robotics_Udacity/projects/catkin_ws_chase_ball/src/av_robot/urdf/robot.xacro (robot description, xacro)
@@ -62,5 +62,5 @@
         </visual>
         <collision name='back_caster_collision'>
-            <origin xyz="-0.3 0 -0.05" rpy=" 0 0 0"/>
+            <origin xyz="-0.3 0 -0.1" rpy=" 0 0 0"/>
             <geometry>
                 <sphere radius="0.099"/>
